File: dedicated_hw/rp2350.kicad_sch (KiCad schematic)
At the start: 28 parts, among them U1 RP2350A, U2 W25Q128JVS, Y1 12MHz

Commit message: Started revising 0.1.0 bugs
Parts:
- added R4: 27, Resistor_SMD:R_0402_1005Metric, symbol Device:R
- C26: footprint Capacitor_SMD:C_0402_1005Metric -> Capacitor_SMD:C_0603_1608Metric
- C35: footprint Capacitor_SMD:C_0402_1005Metric -> Capacitor_SMD:C_0603_1608Metric; LCSC C23733 -> C19666; LCSC Part # C23733 -> C19666
- C36: value 100nF -> 4.7uF; LCSC C307331 -> C23733; LCSC Part # C307331 -> C23733
Connections:
- net +3V3: now also R4.2; no longer C36.1, U1.46 (VREG_AVDD)
- new net: C36.1, R4.1, U1.46 (VREG_AVDD)
Changed lines of the file:
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@@
   (title_block
     (title "Dedicated HW for picoX7")
-    (date "2025-02-04")
-    (rev "0.1.0a")
+    (date "2025-03-04")
+    (rev "0.1.1a")
     (company "https://github.com/GeorgeRudolf/picoX7")
   )
@@
   (junction (at 119.38 33.02) (diameter 0) (color 0 0 0 0)
   )
+  (junction (at 35.56 203.2) (diameter 0) (color 0 0 0 0)
+  )
+  (junction (at 45.72 100.33) (diameter 0) (color 0 0 0 0)
+  )
+  (junction (at 48.26 43.18) (diameter 0) (color 0 0 0 0)
+  )
+  (junction (at 69.85 203.2) (diameter 0) (color 0 0 0 0)
+  )
+  (junction (at 45.72 97.79) (diameter 0) (color 0 0 0 0)
+  )
+  (junction (at 127 33.02) (diameter 0) (color 0 0 0 0)
+  )
   (junction (at 76.2 30.48) (diameter 0) (color 0 0 0 0)
-  )
-  (junction (at 35.56 203.2) (diameter 0) (color 0 0 0 0)
-  )
-  (junction (at 45.72 100.33) (diameter 0) (color 0 0 0 0)
-  )
-  (junction (at 48.26 43.18) (diameter 0) (color 0 0 0 0)
-  )
-  (junction (at 69.85 203.2) (diameter 0) (color 0 0 0 0)
-  )
-  (junction (at 45.72 97.79) (diameter 0) (color 0 0 0 0)
-  )
-  (junction (at 127 33.02) (diameter 0) (color 0 0 0 0)
   )
   (junction (at 39.37 157.48) (diameter 0) (color 0 0 0 0)
@@
     (stroke (width 0) (type default))
   )
+  (wire (pts (xy 74.93 30.48) (xy 76.2 30.48))
+    (stroke (width 0) (type default))
+  )
   (wire (pts (xy 49.53 92.71) (xy 49.53 100.33))
     (stroke (width 0) (type default))
@@
     (stroke (width 0) (type default))
   )
+  (wire (pts (xy 66.04 29.21) (xy 66.04 30.48))
+    (stroke (width 0) (type default))
+  )
   (wire (pts (xy 57.15 53.34) (xy 88.9 53.34))
     (stroke (width 0) (type default))
@@
     (stroke (width 0) (type default))
   )
-  (wire (pts (xy 76.2 29.21) (xy 76.2 30.48))
-    (stroke (width 0) (type default))
-  )
   (wire (pts (xy 27.94 97.79) (xy 27.94 100.33))
     (stroke (width 0) (type default))
@@
   )
   (wire (pts (xy 152.4 95.25) (xy 165.1 95.25))
+    (stroke (width 0) (type default))
+  )
+  (wire (pts (xy 66.04 30.48) (xy 67.31 30.48))
     (stroke (width 0) (type default))
   )
@@
       (effects (font (size 1 1)) (justify left))
     )
-    (property "Value" "100nF" (at 79.121 36.703 0)
+    (property "Value" "4.7uF" (at 79.121 36.703 0)
       (effects (font (size 1 1)) (justify left))
     )
@@
       (effects (font (size 1 1)) hide)
     )
-    (property "LCSC Part #" "C307331" (at 76.2 35.56 0)
-      (effects (font (size 1 1)) hide)
-    )
-    (property "LCSC" "C307331" (at 76.2 35.56 0)
+    (property "LCSC Part #" "C23733" (at 76.2 35.56 0)
+      (effects (font (size 1 1)) hide)
+    )
+    (property "LCSC" "C23733" (at 76.2 35.56 0)
       (effects (font (size 1 1)) hide)
     )
@@
     )
   )
+  (symbol (lib_id "Device:R") (at 71.12 30.48 270) (unit 1)
+    (in_bom yes) (on_board yes) (dnp no)
+    (property "Reference" "R4" (at 71.12 33.02 90)
+      (effects (font (size 1 1)))
+    )
+    (property "Value" "27" (at 71.12 30.48 90)
+      (effects (font (size 1 1)))
+    )
+    (property "Footprint" "Resistor_SMD:R_0402_1005Metric" (at 71.12 28.702 90)
+      (effects (font (size 1 1)) hide)
+    )
+    (property "Datasheet" "~" (at 71.12 30.48 0)
+      (effects (font (size 1 1)) hide)
+    )
+    (property "LCSC" "C25092" (at 71.12 30.48 0)
+      (effects (font (size 1 1)) hide)
+    )
+    (property "LCSC Part #" "C25092" (at 71.12 30.48 0)
+      (effects (font (size 1 1)) hide)
+    )
+    (pin "1")
+    (pin "2")
+    (instances
+      (project "RP2040_minimal"
+        (path "/64357f9c-1097-40ff-93cb-cb8bdaae34cb"
+          (reference "R4") (unit 1)
+        )
+      )
+      (project "gbscsi2"
+        (path "/81c2a5db-c508-405c-87d7-d49be9ddd5e4"
+          (reference "R49") (unit 1)
+        )
+      )
+      (project "picoX7"
+        (path "/8dd66cb3-bd85-43a0-9ef0-1bd8a27e677c/cd18800e-5708-4993-aba3-c5a573d89498"
+          (reference "R35") (unit 1)
+        )
+      )
+    )
+  )
   (symbol (lib_id "Device:C") (at 48.26 48.26 0) (unit 1)
     (in_bom yes) (on_board yes) (dnp no) (fields_autoplaced)
@@
       (effects (font (size 1 1)) (justify left))
     )
-    (property "Footprint" "Capacitor_SMD:C_0402_1005Metric" (at 49.2252 52.07 0)
+    (property "Footprint" "Capacitor_SMD:C_0603_1608Metric" (at 49.2252 52.07 0)
       (effects (font (size 1 1)) hide)
     )
@@
       (effects (font (size 1 1)) hide)
     )
-    (property "LCSC Part #" "C23733" (at 48.26 48.26 0)
-      (effects (font (size 1 1)) hide)
-    )
-    (property "LCSC" "C23733" (at 48.26 48.26 0)
+    (property "LCSC Part #" "C19666" (at 48.26 48.26 0)
+      (effects (font (size 1 1)) hide)
+    )
+    (property "LCSC" "C19666" (at 48.26 48.26 0)
       (effects (font (size 1 1)) hide)
     )
@@
         (path "/8dd66cb3-bd85-43a0-9ef0-1bd8a27e677c/cd18800e-5708-4993-aba3-c5a573d89498"
           (reference "#PWR016") (unit 1)
-        )
-      )
-    )
-  )
-  (symbol (lib_id "power:+3V3") (at 76.2 29.21 0) (unit 1)
-    (in_bom yes) (on_board yes) (dnp no)
-    (property "Reference" "#PWR099" (at 76.2 33.02 0)
-      (effects (font (size 1 1)) hide)
-    )
-    (property "Value" "+3V3" (at 76.581 24.8158 0)
-      (effects (font (size 1 1)))
-    )
-    (property "Footprint" "" (at 76.2 29.21 0)
-      (effects (font (size 1 1)) hide)
-    )
-    (property "Datasheet" "" (at 76.2 29.21 0)
-      (effects (font (size 1 1)) hide)
-    )
-    (pin "1")
-    (instances
-      (project "gbscsi2"
-        (path "/81c2a5db-c508-405c-87d7-d49be9ddd5e4"
-          (reference "#PWR099") (unit 1)
-        )
-      )
-      (project "picoX7"
-        (path "/8dd66cb3-bd85-43a0-9ef0-1bd8a27e677c/cd18800e-5708-4993-aba3-c5a573d89498"
-          (reference "#PWR010") (unit 1)
-        )
-      )
-      (project "RP2350_60QFN_minimal"
-        (path "/94683f5c-9cd9-448e-be96-9792537b5cb8"
-          (reference "#PWR0103") (unit 1)
         )
       )
@@
       (effects (font (size 1 1)) (justify left))
     )
-    (property "Footprint" "Capacitor_SMD:C_0402_1005Metric" (at 37.7952 52.07 0)
+    (property "Footprint" "Capacitor_SMD:C_0603_1608Metric" (at 37.7952 52.07 0)
       (effects (font (size 1 1)) hide)
     )
@@
         )
       )
+    )
+  )
+  (symbol (lib_id "power:+3V3") (at 66.04 29.21 0) (unit 1)
+    (in_bom yes) (on_board yes) (dnp no)
+    (property "Reference" "#PWR099" (at 66.04 33.02 0)
+      (effects (font (size 1 1)) hide)
+    )
+    (property "Value" "+3V3" (at 66.421 24.8158 0)
+      (effects (font (size 1 1)))
+    )
+    (property "Footprint" "" (at 66.04 29.21 0)
+      (effects (font (size 1 1)) hide)
+    )
+    (property "Datasheet" "" (at 66.04 29.21 0)
+      (effects (font (size 1 1)) hide)
+    )
+    (pin "1")
+    (instances
+      (project "gbscsi2"
+        (path "/81c2a5db-c508-405c-87d7-d49be9ddd5e4"
+          (reference "#PWR099") (unit 1)
+        )
+      )
+      (project "picoX7"
+        (path "/8dd66cb3-bd85-43a0-9ef0-1bd8a27e677c/cd18800e-5708-4993-aba3-c5a573d89498"
+          (reference "#PWR010") (unit 1)
+        )
+      )
+      (project "RP2350_60QFN_minimal"
+        (path "/94683f5c-9cd9-448e-be96-9792537b5cb8"
+          (reference "#PWR0103") (unit 1)
+        )
+      )
