File: dedicated_hw/io_pwr.kicad_sch (KiCad schematic)
At the start: 27 parts, among them J1 MIDI in, J1 USB_DATA, J2 Conn_01x03, J2 TF003, J7 Conn_01x04, U3 H11L1, U6 AMS1117-3.3, U9 USB TVS

Commit message: Started revising 0.1.0 bugs
Parts:
- added R? (x3): 10k, Resistor_SMD:R_0402_1005Metric, symbol zuluscsi-rescue:R
Connections:
- net +3V3: now also R?.2, R?.2, R?.2
- net SD_CLK: now also R?.1
- net SD_MISO: now also R?.1
- net SD_MOSI: now also R?.1
Changed lines of the file:
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@@
   (junction (at 60.96 220.98) (diameter 0) (color 0 0 0 0)
   )
+  (junction (at 143.51 207.01) (diameter 0) (color 0 0 0 0)
+  )
+  (junction (at 153.67 231.14) (diameter 0) (color 0 0 0 0)
+  )
+  (junction (at 148.59 207.01) (diameter 0) (color 0 0 0 0)
+  )
   (junction (at 66.04 50.8) (diameter 0.9144) (color 0 0 0 0)
   )
@@
   (junction (at 123.19 241.3) (diameter 0) (color 0 0 0 0)
   )
+  (junction (at 148.59 226.06) (diameter 0) (color 0 0 0 0)
+  )
   (junction (at 81.28 184.15) (diameter 0) (color 0 0 0 0)
   )
@@
   )
   (junction (at 123.19 223.52) (diameter 0) (color 0 0 0 0)
+  )
+  (junction (at 143.51 220.98) (diameter 0) (color 0 0 0 0)
   )
   (junction (at 185.42 223.52) (diameter 0) (color 0 0 0 0)
@@
     (stroke (width 0) (type default))
   )
+  (wire (pts (xy 148.59 214.63) (xy 148.59 226.06))
+    (stroke (width 0) (type default))
+  )
   (wire (pts (xy 158.75 55.88) (xy 152.4 55.88))
+    (stroke (width 0) (type default))
+  )
+  (wire (pts (xy 148.59 226.06) (xy 158.75 226.06))
     (stroke (width 0) (type default))
   )
@@
     (stroke (width 0) (type default))
   )
+  (wire (pts (xy 153.67 231.14) (xy 158.75 231.14))
+    (stroke (width 0) (type default))
+  )
   (wire (pts (xy 151.13 177.8) (xy 154.94 177.8))
     (stroke (width 0) (type default))
   )
-  (wire (pts (xy 135.89 226.06) (xy 158.75 226.06))
+  (wire (pts (xy 135.89 226.06) (xy 148.59 226.06))
     (stroke (width 0) (type default))
   )
@@
     (stroke (width 0) (type solid))
   )
-  (wire (pts (xy 135.89 231.14) (xy 158.75 231.14))
+  (wire (pts (xy 135.89 231.14) (xy 153.67 231.14))
     (stroke (width 0) (type default))
   )
@@
     (stroke (width 0) (type solid))
   )
-  (wire (pts (xy 135.89 220.98) (xy 158.75 220.98))
+  (wire (pts (xy 135.89 220.98) (xy 143.51 220.98))
+    (stroke (width 0) (type default))
+  )
+  (wire (pts (xy 143.51 207.01) (xy 148.59 207.01))
+    (stroke (width 0) (type default))
+  )
+  (wire (pts (xy 143.51 220.98) (xy 158.75 220.98))
     (stroke (width 0) (type default))
   )
@@
     (stroke (width 0) (type default))
   )
+  (wire (pts (xy 153.67 214.63) (xy 153.67 231.14))
+    (stroke (width 0) (type default))
+  )
   (wire (pts (xy 40.64 82.55) (xy 48.26 82.55))
     (stroke (width 0) (type solid))
@@
     (stroke (width 0) (type default))
   )
+  (wire (pts (xy 148.59 207.01) (xy 153.67 207.01))
+    (stroke (width 0) (type default))
+  )
+  (wire (pts (xy 143.51 205.74) (xy 143.51 207.01))
+    (stroke (width 0) (type default))
+  )
   (wire (pts (xy 158.75 223.52) (xy 123.19 223.52))
     (stroke (width 0) (type default))
@@
   )
   (wire (pts (xy 81.28 220.98) (xy 81.28 218.44))
+    (stroke (width 0) (type default))
+  )
+  (wire (pts (xy 143.51 214.63) (xy 143.51 220.98))
     (stroke (width 0) (type default))
   )
@@
     )
   )
+  (symbol (lib_id "power:+3.3V") (at 143.51 205.74 0) (unit 1)
+    (in_bom yes) (on_board yes) (dnp no) (fields_autoplaced)
+    (property "Reference" "#PWR03" (at 143.51 209.55 0)
+      (effects (font (size 1 1)) hide)
+    )
+    (property "Value" "+3.3V" (at 143.51 200.66 0)
+      (effects (font (size 1 1)))
+    )
+    (property "Footprint" "" (at 143.51 205.74 0)
+      (effects (font (size 1 1)) hide)
+    )
+    (property "Datasheet" "" (at 143.51 205.74 0)
+      (effects (font (size 1 1)) hide)
+    )
+    (pin "1")
+    (instances
+      (project "gbscsi2"
+        (path "/81c2a5db-c508-405c-87d7-d49be9ddd5e4"
+          (reference "#PWR03") (unit 1)
+        )
+      )
+      (project "picoX7"
+        (path "/8dd66cb3-bd85-43a0-9ef0-1bd8a27e677c/cd18800e-5708-4993-aba3-c5a573d89498"
+          (reference "#PWR092") (unit 1)
+        )
+        (path "/8dd66cb3-bd85-43a0-9ef0-1bd8a27e677c/6b679a71-01f9-4bb3-b0ed-858fef2e27bb"
+          (reference "#PWR0108") (unit 1)
+        )
+      )
+    )
+  )
   (symbol (lib_id "Device:C_Small") (at 127 143.51 0) (unit 1)
     (in_bom yes) (on_board yes) (dnp no)
@@
         (path "/8dd66cb3-bd85-43a0-9ef0-1bd8a27e677c/6b679a71-01f9-4bb3-b0ed-858fef2e27bb"
           (reference "C25") (unit 1)
+        )
+      )
+    )
+  )
+  (symbol (lib_id "zuluscsi-rescue:R") (at 153.67 210.82 180) (unit 1)
+    (in_bom yes) (on_board yes) (dnp no)
+    (property "Reference" "R?" (at 151.638 210.82 90)
+      (effects (font (size 1 1)))
+    )
+    (property "Value" "10k" (at 153.67 210.82 90)
+      (effects (font (size 1 1)))
+    )
+    (property "Footprint" "Resistor_SMD:R_0402_1005Metric" (at 155.448 210.82 90)
+      (effects (font (size 1 1)) hide)
+    )
+    (property "Datasheet" "" (at 153.67 210.82 0)
+      (effects (font (size 1 1)))
+    )
+    (property "LCSC" "C25744" (at 153.67 210.82 0)
+      (effects (font (size 1 1)) hide)
+    )
+    (property "LCSC Part #" "C25744" (at 153.67 210.82 0)
+      (effects (font (size 1 1)) hide)
+    )
+    (pin "1")
+    (pin "2")
+    (instances
+      (project "ZuluSCSI-Pico-OSHW"
+        (path "/0a1a4d88-972a-46ce-b25e-6cb796bd41f7/00000000-0000-0000-0000-000055ff7cc4"
+          (reference "R?") (unit 1)
+        )
+      )
+      (project "cpu"
+        (path "/45b7fe01-a2fa-40c2-a3a2-4a9ae7c34dba"
+          (reference "R?") (unit 1)
+        )
+      )
+      (project "gbscsi2"
+        (path "/81c2a5db-c508-405c-87d7-d49be9ddd5e4"
+          (reference "R1") (unit 1)
+        )
+      )
+      (project "picoX7"
+        (path "/8dd66cb3-bd85-43a0-9ef0-1bd8a27e677c/cd18800e-5708-4993-aba3-c5a573d89498"
+          (reference "R29") (unit 1)
+        )
+        (path "/8dd66cb3-bd85-43a0-9ef0-1bd8a27e677c/6b679a71-01f9-4bb3-b0ed-858fef2e27bb"
+          (reference "R33") (unit 1)
         )
       )
@@
         (path "/ea7c53f9-3aa8-4198-9879-de95a5257915"
           (reference "#PWR?") (unit 1)
+        )
+      )
+    )
+  )
+  (symbol (lib_id "zuluscsi-rescue:R") (at 148.59 210.82 180) (unit 1)
+    (in_bom yes) (on_board yes) (dnp no)
+    (property "Reference" "R?" (at 146.558 210.82 90)
+      (effects (font (size 1 1)))
+    )
+    (property "Value" "10k" (at 148.59 210.82 90)
+      (effects (font (size 1 1)))
+    )
+    (property "Footprint" "Resistor_SMD:R_0402_1005Metric" (at 150.368 210.82 90)
+      (effects (font (size 1 1)) hide)
+    )
+    (property "Datasheet" "" (at 148.59 210.82 0)
+      (effects (font (size 1 1)))
+    )
+    (property "LCSC" "C25744" (at 148.59 210.82 0)
+      (effects (font (size 1 1)) hide)
+    )
+    (property "LCSC Part #" "C25744" (at 148.59 210.82 0)
+      (effects (font (size 1 1)) hide)
+    )
+    (pin "1")
+    (pin "2")
+    (instances
+      (project "ZuluSCSI-Pico-OSHW"
+        (path "/0a1a4d88-972a-46ce-b25e-6cb796bd41f7/00000000-0000-0000-0000-000055ff7cc4"
+          (reference "R?") (unit 1)
+        )
+      )
+      (project "cpu"
+        (path "/45b7fe01-a2fa-40c2-a3a2-4a9ae7c34dba"
+          (reference "R?") (unit 1)
+        )
+      )
+      (project "gbscsi2"
+        (path "/81c2a5db-c508-405c-87d7-d49be9ddd5e4"
+          (reference "R1") (unit 1)
+        )
+      )
+      (project "picoX7"
+        (path "/8dd66cb3-bd85-43a0-9ef0-1bd8a27e677c/cd18800e-5708-4993-aba3-c5a573d89498"
+          (reference "R29") (unit 1)
+        )
+        (path "/8dd66cb3-bd85-43a0-9ef0-1bd8a27e677c/6b679a71-01f9-4bb3-b0ed-858fef2e27bb"
+          (reference "R32") (unit 1)
         )
       )
@@
         )
       )
+    )
+  )
+  (symbol (lib_id "zuluscsi-rescue:R") (at 143.51 210.82 180) (unit 1)
+    (in_bom yes) (on_board yes) (dnp no)
+    (property "Reference" "R?" (at 141.478 210.82 90)
+      (effects (font (size 1 1)))
+    )
+    (property "Value" "10k" (at 143.51 210.82 90)
+      (effects (font (size 1 1)))
+    )
+    (property "Footprint" "Resistor_SMD:R_0402_1005Metric" (at 145.288 210.82 90)
+      (effects (font (size 1 1)) hide)
+    )
+    (property "Datasheet" "" (at 143.51 210.82 0)
+      (effects (font (size 1 1)))
+    )
+    (property "LCSC" "C25744" (at 143.51 210.82 0)
+      (effects (font (size 1 1)) hide)
+    )
+    (property "LCSC Part #" "C25744" (at 143.51 210.82 0)
+      (effects (font (size 1 1)) hide)
+    )
+    (pin "1")
+    (pin "2")
+    (instances
+      (project "ZuluSCSI-Pico-OSHW"
+        (path "/0a1a4d88-972a-46ce-b25e-6cb796bd41f7/00000000-0000-0000-0000-000055ff7cc4"
+          (reference "R?") (unit 1)
+        )
+      )
+      (project "cpu"
+        (path "/45b7fe01-a2fa-40c2-a3a2-4a9ae7c34dba"
+          (reference "R?") (unit 1)
+        )
+      )
+      (project "gbscsi2"
+        (path "/81c2a5db-c508-405c-87d7-d49be9ddd5e4"
+          (reference "R1") (unit 1)
+        )
+      )
+      (project "picoX7"
+        (path "/8dd66cb3-bd85-43a0-9ef0-1bd8a27e677c/cd18800e-5708-4993-aba3-c5a573d89498"
+          (reference "R29") (unit 1)
+        )
+        (path "/8dd66cb3-bd85-43a0-9ef0-1bd8a27e677c/6b679a71-01f9-4bb3-b0ed-858fef2e27bb"
+          (reference "R31") (unit 1)
+        )
+      )

Commit message: Slowly sorting out 0.1.0 bugs
Parts:
- removed C19: 4.7nF, Capacitor_SMD:C_0402_1005Metric, symbol Device:C_Small
- removed R?: 1M, Resistor_SMD:R_0402_1005Metric, symbol Device:R
- C1: value 100nF -> 4.7uF; LCSC C307331 -> C23733; LCSC Part # C307331 -> C23733
Connections:
- net GND: now also J1.S1 (SHIELD)
Changed lines of the file:
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@@
   (junction (at 123.19 228.6) (diameter 0) (color 0 0 0 0)
   )
-  (junction (at 40.64 82.55) (diameter 0) (color 0 0 0 0)
-  )
   (junction (at 151.13 177.8) (diameter 0) (color 0 0 0 0)
   )
@@
   (junction (at 185.42 226.06) (diameter 0) (color 0 0 0 0)
   )
+  (junction (at 48.26 71.12) (diameter 0) (color 0 0 0 0)
+  )
   (junction (at 90.17 52.07) (diameter 0) (color 0 0 0 0)
   )
@@
   )
   (junction (at 151.13 170.18) (diameter 0) (color 0 0 0 0)
-  )
-  (junction (at 40.64 74.93) (diameter 0) (color 0 0 0 0)
   )
   (junction (at 66.04 48.26) (diameter 0.9144) (color 0 0 0 0)
@@
     (stroke (width 0) (type solid))
   )
+  (wire (pts (xy 40.64 71.12) (xy 48.26 71.12))
+    (stroke (width 0) (type default))
+  )
   (wire (pts (xy 63.5 50.8) (xy 66.04 50.8))
     (stroke (width 0) (type solid))
@@
     (stroke (width 0) (type default))
   )
-  (wire (pts (xy 40.64 81.28) (xy 40.64 82.55))
-    (stroke (width 0) (type solid))
-  )
   (wire (pts (xy 154.94 35.56) (xy 142.24 35.56))
     (stroke (width 0) (type default))
@@
     (stroke (width 0) (type default))
   )
-  (wire (pts (xy 40.64 71.12) (xy 40.64 74.93))
-    (stroke (width 0) (type default))
-  )
   (wire (pts (xy 66.04 48.26) (xy 63.5 48.26))
     (stroke (width 0) (type solid))
@@
     (stroke (width 0) (type default))
   )
-  (wire (pts (xy 40.64 74.93) (xy 40.64 76.2))
-    (stroke (width 0) (type solid))
-  )
   (wire (pts (xy 138.43 241.3) (xy 123.19 241.3))
     (stroke (width 0) (type default))
@@
     (stroke (width 0) (type default))
   )
-  (wire (pts (xy 40.64 82.55) (xy 48.26 82.55))
-    (stroke (width 0) (type solid))
-  )
   (wire (pts (xy 138.43 233.68) (xy 138.43 218.44))
     (stroke (width 0) (type default))
-  )
-  (wire (pts (xy 36.83 82.55) (xy 40.64 82.55))
-    (stroke (width 0) (type solid))
-  )
-  (wire (pts (xy 36.83 74.93) (xy 40.64 74.93))
-    (stroke (width 0) (type solid))
   )
   (wire (pts (xy 66.04 48.26) (xy 69.85 48.26))
@@
         (path "/94683f5c-9cd9-448e-be96-9792537b5cb8"
           (reference "#PWR0106") (unit 1)
-        )
-      )
-    )
-  )
-  (symbol (lib_id "Device:C_Small") (at 40.64 78.74 0) (mirror y) (unit 1)
-    (in_bom yes) (on_board yes) (dnp no)
-    (property "Reference" "C19" (at 44.45 76.2 0)
-      (effects (font (size 1 1)) (justify left))
-    )
-    (property "Value" "4.7nF" (at 46.99 81.28 0)
-      (effects (font (size 1 1)) (justify left))
-    )
-    (property "Footprint" "Capacitor_SMD:C_0402_1005Metric" (at 40.64 78.74 0)
-      (effects (font (size 1 1)) hide)
-    )
-    (property "Datasheet" "~" (at 40.64 78.74 0)
-      (effects (font (size 1 1)) hide)
-    )
-    (property "LCSC" "C1538" (at 40.64 78.74 0)
-      (effects (font (size 1 1)) hide)
-    )
-    (property "LCSC Part #" "C1538" (at 40.64 78.74 0)
-      (effects (font (size 1 1)) hide)
-    )
-    (pin "1")
-    (pin "2")
-    (instances
-      (project "gbscsi2"
-        (path "/81c2a5db-c508-405c-87d7-d49be9ddd5e4"
-          (reference "C19") (unit 1)
-        )
-      )
-      (project "poe_hat_v1.4.2"
-        (path "/84fe1d92-0d61-4eda-acb4-e2fc63573041"
-          (reference "C8") (unit 1)
-        )
-      )
-      (project "picoX7"
-        (path "/8dd66cb3-bd85-43a0-9ef0-1bd8a27e677c/6b679a71-01f9-4bb3-b0ed-858fef2e27bb"
-          (reference "C17") (unit 1)
         )
       )
@@
       (effects (font (size 1 1)))
     )
-    (property "Value" "100nF" (at 118.11 227.33 0)
+    (property "Value" "4.7uF" (at 118.11 227.33 0)
       (effects (font (size 1 1)))
     )
@@
       (effects (font (size 1 1)) hide)
     )
-    (property "LCSC" "C307331" (at 123.19 226.06 0)
-      (effects (font (size 1 1)) hide)
-    )
-    (property "LCSC Part #" "C307331" (at 123.19 226.06 0)
+    (property "LCSC" "C23733" (at 123.19 226.06 0)
+      (effects (font (size 1 1)) hide)
+    )
+    (property "LCSC Part #" "C23733" (at 123.19 226.06 0)
       (effects (font (size 1.27 1.27)) hide)
     )
@@
         )
       )
-    )
-  )
-  (symbol (lib_id "Device:R") (at 36.83 78.74 0) (mirror y) (unit 1)
-    (in_bom yes) (on_board yes) (dnp no)
-    (property "Reference" "R?" (at 34.29 78.74 90)
-      (effects (font (size 1 1)))
-    )
-    (property "Value" "1M" (at 36.83 78.74 90)
-      (effects (font (size 1 1)))
-    )
-    (property "Footprint" "Resistor_SMD:R_0402_1005Metric" (at 38.608 78.74 90)
-      (effects (font (size 1 1)) hide)
-    )
-    (property "Datasheet" "~" (at 36.83 78.74 0)
-      (effects (font (size 1 1)) hide)
-    )
-    (property "LCSC" "C26083" (at 36.83 78.74 0)
-      (effects (font (size 1 1)) hide)
-    )
-    (property "LCSC Part #" "C26083" (at 36.83 78.74 0)
-      (effects (font (size 1 1)) hide)
-    )
-    (pin "1")
-    (pin "2")
-    (instances
-      (project "ZuluSCSI-Pico-OSHW"
-        (path "/0a1a4d88-972a-46ce-b25e-6cb796bd41f7/00000000-0000-0000-0000-000055ff7cc4"
-          (reference "R?") (unit 1)
-        )
-      )
-      (project "cpu"
-        (path "/45b7fe01-a2fa-40c2-a3a2-4a9ae7c34dba"
-          (reference "R?") (unit 1)
-        )
-      )
-      (project "gbscsi2"
-        (path "/81c2a5db-c508-405c-87d7-d49be9ddd5e4"
-          (reference "R15") (unit 1)
-        )
-      )
-      (project "picoX7"
-        (path "/8dd66cb3-bd85-43a0-9ef0-1bd8a27e677c/6b679a71-01f9-4bb3-b0ed-858fef2e27bb"
-          (reference "R6") (unit 1)
-        )
-      )
