File: dedicated_hw/picoX7.kicad_pcb (KiCad board)
At the start: 4 copper layers, 90.7 x 65.4 mm, 110 parts, among them J1 Conn_01x04, J2 Conn_01x03, J3 USB_DATA, J4 MIDI in, J5 PJ-320-3P SMT, J6 Conn_01x03, J7 Conn_01x03, J8 TF003, SW1 SW_SPST, SW2 SW_SPST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

Commit message: Started revising 0.1.0 bugs
Parts:
- added R31: 10k, Resistor_SMD:R_0402_1005Metric, F.Cu at (149.4, 46.0)
- added R32: 10k, Resistor_SMD:R_0402_1005Metric, F.Cu at (151.6, 46.5)
- added R33: 10k, Resistor_SMD:R_0402_1005Metric, F.Cu at (153.9, 46.0)
- added R35: 27, Resistor_SMD:R_0402_1005Metric, F.Cu at (111.5, 49.5)
- C4, C5: footprint Capacitor_SMD:C_0402_1005Metric -> Capacitor_SMD:C_0603_1608Metric
- C6: value 100nF -> 4.7uF
- moved C6 1.34 mm to (111.5, 50.7), turned to 180 degrees
- moved L1 1.34 mm to (107.3, 52.1)
- moved C5 0.91 mm to (109.6, 53.1)
- moved C4 0.54 mm to (111.1, 53.1)
- moved C42 0.16 mm to (151.6, 45.3)
Connections:
- C6 pad 1: +3V3 -> Net-(U1-VREG_AVDD)
- U1 pad 46: +3V3 -> Net-(U1-VREG_AVDD)
Routing:
- net +3V3: track 358.4 -> 365.5 mm
- net Net-(U1-VREG_AVDD): track 0.00 -> 4.50 mm
- net /RP2350 Core/SD_CLK: track 56.4 -> 58.8 mm
- net /RP2350 Core/VREG_LX: track 4.94 -> 7.17 mm
- net +1V1: track 29.3 -> 30.8 mm
- net /RP2350 Core/SD_MISO: track 62.1 -> 63.3 mm
- net /RP2350 Core/SD_MOSI: track 59.6 -> 60.8 mm
Other:
- board text added: "PCB v0.1.1b"
- board text removed: "PCB v0.1.0b"

Commit message: Slowly sorting out 0.1.0 bugs
Parts:
- removed C17: 4.7nF, Capacitor_SMD:C_0402_1005Metric
- removed R6: 1M, Resistor_SMD:R_0402_1005Metric
- C42: value 100nF -> 4.7uF
Connections:
- J3 pad S1: Net-(J3-SHIELD) -> GND
Routing:
- net Net-(J3-SHIELD): track 21.8 -> 0.00 mm
